Commit message: add config change laser frame

File: pal_description_package/pal_description_package/urdf/pal_description_package.urdf (robot description, URDF)
Before this commit: robot pal_description_package, 8 links, 7 joints
Links:
- removed link laser_link
- added link laser_frame, mass 0.14299; collision mesh filename=package://pal_description_package/meshes/laser_link.STL; visual mesh filename=package://pal_description_package/meshes/laser_link.STL
Joints:
- joint base_to_laser_link: child laser_link -> laser_frame

Commit message: laser_changed_pos

File: pal_description_package/pal_description_package/urdf/pal_description_package.urdf (robot description, URDF)
Before this commit: robot pal_description_package, 8 links, 7 joints
Links:
- removed link laser_frame
- added link laser_link, mass 0.14299; collision mesh filename=package://pal_description_package/meshes/laser_link.STL; visual mesh filename=package://pal_description_package/meshes/laser_link.STL
Joints:
- joint base_to_laser_link: child laser_frame -> laser_link
